File: imu_geolocator.kicad_pcb (KiCad board)
At the start: 4 copper layers, 57 parts, among them IC1 CG2214M6-C2, J1 Conn_01x05_Pin, J2 Conn_01x08_Pin, J3 A-1JB, Q1 PMOS, U1 STM32WLE5C8Ux, U2 TPS62202DBV, U3 ICM-42688-P, U4 AK09918C

Commit message: Routing in progress
Parts:
- removed L3: 10u, Inductor_SMD:L_0603_1608Metric
- added FB1: FerriteBead, Inductor_SMD:L_0603_1608Metric, F.Cu at (95.5, 74.4)
- added R7: 10K, Resistor_SMD:R_0603_1608Metric, F.Cu at (97.0, 69.4)
- added R8: 10K, Resistor_SMD:R_0603_1608Metric, F.Cu at (98.8, 69.4)
- B1: moved to B.Cu
- L1, L2: footprint Inductor_SMD:L_0603_1608Metric -> Inductor_SMD:L_0805_2012Metric
- moved J1 83.8 mm to (111.8, 77.5), turned to 180 degrees
- moved C9 83.5 mm to (102.7, 77.5), turned to 90 degrees
- moved F1 82.8 mm to (105.7, 81.3), turned to 180 degrees
- moved R2 81.9 mm to (107.5, 76.8), turned to 90 degrees
- moved C11 81.3 mm to (105.2, 70.4)
- moved C12 81.1 mm to (105.2, 72.2)
- moved C13 80.8 mm to (105.2, 73.9)
- moved C8 77.9 mm to (99.4, 76.6)
- moved C10 76.8 mm to (98.3, 73.6), turned to 180 degrees
- moved B1 71.7 mm to (91.0, 72.3), turned to 180 degrees
- moved L2 71.4 mm to (95.9, 79.2), turned to 90 degrees
- moved L5 67.1 mm to (43.7, 85.5), turned to 90 degrees
- moved D1 66.3 mm to (108.4, 80.5), turned to -90 degrees
- moved J3 65.7 mm to (34.1, 76.4), turned to -90 degrees
- moved D2 64.8 mm to (105.2, 78.1), turned to -90 degrees
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Connections:
- R6 pad 1: VCC -> VDD
- U1 pad 12: unconnected-(U1-PA4-Pad12) -> /MCU_FSYNC
- U1 pad 13: /MCU_FSYNC -> /IMU_INT
- U1 pad 37: VCC -> VDD
Routing:
- net GND: track 0.00 -> 69.2 mm, vias 0 -> 23
- net /MCU_LED_R: track 0.00 -> 40.0 mm, vias 0 -> 2
- net VDD: track 0.00 -> 39.9 mm, vias 0 -> 10
- net /MCU_LED_G: track 0.00 -> 33.8 mm, vias 0 -> 2
- net /RF_CTRL: track 0.00 -> 31.2 mm, vias 0 -> 3
- net /MCU_LED_B: track 0.00 -> 31.1 mm, vias 0 -> 2
- net /VR_PA: track 0.00 -> 29.2 mm, vias 0 -> 2
- net /RFO_HP: track 0.00 -> 23.4 mm, vias 0 -> 2
- net /VDDRF1V55: track 0.00 -> 21.4 mm, vias 0 -> 3
- net /RF_nCTRL: track 0.00 -> 16.2 mm, vias 0 -> 2
- net /LED_B: track 0.00 -> 15.0 mm, vias 0 -> 2
- net /RFI_P: track 0.00 -> 11.4 mm, vias 0 -> 2
- net +3V3: track 0.00 -> 10.8 mm
- net /RF/RF_RX: track 0.00 -> 9.91 mm
- net VCC: track 0.00 -> 9.31 mm, vias 0 -> 1
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- added copper zone on B.Cu, net +BATT
- added copper zone on B.Cu, net GND
- added copper zone on In1.Cu, net GND
- added copper zone on F.Cu, net VDD
Other:
- board outline added: 50.8 x 48.3 mm

Commit message: Finished routing v0.1
Parts:
- moved J2 76.0 mm to (105.0, 59.7), turned to -90 degrees
- moved R1 66.9 mm to (105.4, 68.4)
- moved L1 34.1 mm to (92.7, 69.3)
- moved C1 33.7 mm to (92.0, 80.1)
- moved C16 33.7 mm to (78.3, 77.7)
- moved C18 33.7 mm to (73.7, 76.8)
- moved C24 33.7 mm to (69.2, 73.2)
- moved C27 33.7 mm to (70.8, 67.2)
- moved L7 33.7 mm to (75.1, 71.7)
- moved L8 33.7 mm to (67.2, 73.3)
- moved R6 33.7 mm to (70.1, 78.9)
- moved C17 33.7 mm to (73.7, 78.6)
- moved C19 33.7 mm to (76.6, 67.0)
- moved C23 33.7 mm to (71.2, 73.3)
- moved C25 33.7 mm to (65.2, 73.3)
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Routing:
- net /NRST: track 2.08 -> 46.3 mm, vias 1 -> 2
- net /SWDIO: track 1.63 -> 40.9 mm
- net /SWCLK: track 1.99 -> 38.7 mm
- net /IMU_INT: track 3.20 -> 37.3 mm
- net VCC: track 9.31 -> 41.5 mm, vias 1 -> 0
- net /SDA: track 6.05 -> 33.1 mm, vias 0 -> 3
- net /MCU_FSYNC: track 2.62 -> 28.6 mm, vias 1 -> 2
- net /SCL: track 7.62 -> 29.0 mm
- net /UART_RX: track 1.62 -> 22.0 mm, vias 1 -> 2
- net /UART_TX: track 2.10 -> 22.2 mm, vias 1 -> 2
- net GND: track 69.2 -> 84.4 mm, vias 23 -> 24
- net VDD: track 39.9 -> 50.7 mm, vias 10 -> 11
- net /RFO_HP: track 23.4 -> 33.7 mm
- net VDDA: track 5.30 -> 13.9 mm, vias 0 -> 2
- net /VR_PA: track 29.2 -> 20.9 mm
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- added copper zone on In2.Cu, net VDD
Other:
- board size 50.8 x 48.3 mm -> 51.1 x 26.9 mm
- board text added: "GND"
- board text added: "IMU Geolocalizer v0.1"
- board text added: "NRST SWDIO SWCLK 3V3 GND"
- board text added: "RX"
- board text added: "SCL"
- board text added: "SDA"
- board text added: "TX"
