File: imu_geolocator.kicad_pcb (KiCad board)
At the start: 4 copper layers, 51.1 x 26.9 mm, 59 parts, among them IC1 CG2214M6-C2, J1 Conn_01x05_Pin, J2 Conn_01x08_Pin, J3 A-1JB, Q1 PMOS, U1 STM32WLE5C8Ux, U2 TPS62202DBV, U3 ICM-42688-P, U4 AK09918C

Commit message: Schematic done
Other:
- board text added: "IMU Geolocator v0.1"
- board text removed: "IMU Geolocalizer v0.1"
Changed lines of the file:
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@@
       (outputformat 1)
       (mirror false)
-      (drillshape 1)
+      (drillshape 0)
       (scaleselection 1)
-      (outputdirectory "")
+      (outputdirectory "output/")
     )
   )
@@
     (fp_line (start 3.5 3.5) (end -3.5 3.5)
       (stroke (width 0.1) (type solid)) (layer "F.Fab"))
-    (pad "" smd roundrect (at -2.1 -2.1 270) (size 1.13 1.13) (layers "F.Paste") (roundrect_rratio 0.221239))
-    (pad "" smd roundrect (at -2.1 -0.7 270) (size 1.13 1.13) (layers "F.Paste") (roundrect_rratio 0.221239))
-    (pad "" smd roundrect (at -2.1 0.7 270) (size 1.13 1.13) (layers "F.Paste") (roundrect_rratio 0.221239))
-    (pad "" smd roundrect (at -2.1 2.1 270) (size 1.13 1.13) (layers "F.Paste") (roundrect_rratio 0.221239))
-    (pad "" smd roundrect (at -0.7 -2.1 270) (size 1.13 1.13) (layers "F.Paste") (roundrect_rratio 0.221239))
-    (pad "" smd roundrect (at -0.7 -0.7 270) (size 1.13 1.13) (layers "F.Paste") (roundrect_rratio 0.221239))
-    (pad "" smd roundrect (at -0.7 0.7 270) (size 1.13 1.13) (layers "F.Paste") (roundrect_rratio 0.221239))
-    (pad "" smd roundrect (at -0.7 2.1 270) (size 1.13 1.13) (layers "F.Paste") (roundrect_rratio 0.221239))
-    (pad "" smd roundrect (at 0.7 -2.1 270) (size 1.13 1.13) (layers "F.Paste") (roundrect_rratio 0.221239))
-    (pad "" smd roundrect (at 0.7 -0.7 270) (size 1.13 1.13) (layers "F.Paste") (roundrect_rratio 0.221239))
-    (pad "" smd roundrect (at 0.7 0.7 270) (size 1.13 1.13) (layers "F.Paste") (roundrect_rratio 0.221239))
-    (pad "" smd roundrect (at 0.7 2.1 270) (size 1.13 1.13) (layers "F.Paste") (roundrect_rratio 0.221239))
-    (pad "" smd roundrect (at 2.1 -2.1 270) (size 1.13 1.13) (layers "F.Paste") (roundrect_rratio 0.221239))
-    (pad "" smd roundrect (at 2.1 -0.7 270) (size 1.13 1.13) (layers "F.Paste") (roundrect_rratio 0.221239))
-    (pad "" smd roundrect (at 2.1 0.7 270) (size 1.13 1.13) (layers "F.Paste") (roundrect_rratio 0.221239))
-    (pad "" smd roundrect (at 2.1 2.1 270) (size 1.13 1.13) (layers "F.Paste") (roundrect_rratio 0.221239))
+    (pad "" smd roundrect (at -2.1 -2.1 270) (size 1.13 1.13) (layers "F.Paste") (roundrect_rratio 0.2212389381))
+    (pad "" smd roundrect (at -2.1 -0.7 270) (size 1.13 1.13) (layers "F.Paste") (roundrect_rratio 0.2212389381))
+    (pad "" smd roundrect (at -2.1 0.7 270) (size 1.13 1.13) (layers "F.Paste") (roundrect_rratio 0.2212389381))
+    (pad "" smd roundrect (at -2.1 2.1 270) (size 1.13 1.13) (layers "F.Paste") (roundrect_rratio 0.2212389381))
+    (pad "" smd roundrect (at -0.7 -2.1 270) (size 1.13 1.13) (layers "F.Paste") (roundrect_rratio 0.2212389381))
+    (pad "" smd roundrect (at -0.7 -0.7 270) (size 1.13 1.13) (layers "F.Paste") (roundrect_rratio 0.2212389381))
+    (pad "" smd roundrect (at -0.7 0.7 270) (size 1.13 1.13) (layers "F.Paste") (roundrect_rratio 0.2212389381))
+    (pad "" smd roundrect (at -0.7 2.1 270) (size 1.13 1.13) (layers "F.Paste") (roundrect_rratio 0.2212389381))
+    (pad "" smd roundrect (at 0.7 -2.1 270) (size 1.13 1.13) (layers "F.Paste") (roundrect_rratio 0.2212389381))
+    (pad "" smd roundrect (at 0.7 -0.7 270) (size 1.13 1.13) (layers "F.Paste") (roundrect_rratio 0.2212389381))
+    (pad "" smd roundrect (at 0.7 0.7 270) (size 1.13 1.13) (layers "F.Paste") (roundrect_rratio 0.2212389381))
+    (pad "" smd roundrect (at 0.7 2.1 270) (size 1.13 1.13) (layers "F.Paste") (roundrect_rratio 0.2212389381))
+    (pad "" smd roundrect (at 2.1 -2.1 270) (size 1.13 1.13) (layers "F.Paste") (roundrect_rratio 0.2212389381))
+    (pad "" smd roundrect (at 2.1 -0.7 270) (size 1.13 1.13) (layers "F.Paste") (roundrect_rratio 0.2212389381))
+    (pad "" smd roundrect (at 2.1 0.7 270) (size 1.13 1.13) (layers "F.Paste") (roundrect_rratio 0.2212389381))
+    (pad "" smd roundrect (at 2.1 2.1 270) (size 1.13 1.13) (layers "F.Paste") (roundrect_rratio 0.2212389381))
     (pad "1" smd roundrect (at -3.4375 -2.75 270) (size 0.875 0.25) (layers "F.Cu" "F.Paste" "F.Mask") (roundrect_rratio 0.25)
       (net 42 "unconnected-(U1-PB3-Pad1)") (pinfunction "PB3") (pintype "bidirectional"))
@@
     (effects (font (size 1 1) (thickness 0.15)) (justify left bottom))
   )
-  (gr_text "IMU Geolocalizer v0.1" (at 62.992 59.182) (layer "F.SilkS")
+  (gr_text "IMU Geolocator v0.1" (at 62.992 59.182) (layer "F.SilkS")
     (effects (font (size 1 1) (thickness 0.15)) (justify left bottom))
   )

Commit message: Routing done
Parts:
- removed the C1 at (92.0, 80.1)
- removed C13: 2.2u, Capacitor_SMD:C_0603_1608Metric
- removed C14: 10n, Capacitor_SMD:C_0603_1608Metric
- removed C15: 47p, Capacitor_SMD:C_0603_1608Metric
- removed C16: 2.4p, Capacitor_SMD:C_0603_1608Metric
- removed C17, C20: 4.7p, Capacitor_SMD:C_0603_1608Metric
- removed C18, C22: 1.8p, Capacitor_SMD:C_0603_1608Metric
- removed C19, C23: 33p, Capacitor_SMD:C_0603_1608Metric
- removed the C2 at (80.4, 67.3)
- removed C21: 1.2p, Capacitor_SMD:C_0603_1608Metric
- removed C24, C25: 3.3p, Capacitor_SMD:C_0603_1608Metric
- removed C26, C27: 1n, Capacitor_SMD:C_0603_1608Metric
- removed the C5 at (92.0, 71.6)
- removed IC1: CG2214M6-C2, CG2214M6-C2:SOTFL48P130X55-6N
- removed J3: A-1JB, A-1JB:AMPHENOL_A-1JB
- removed L2: 10u, Inductor_SMD:L_0805_2012Metric
- removed L4: 33n, Inductor_SMD:L_0603_1608Metric
- removed L5, L6: 10n, Inductor_SMD:L_0603_1608Metric
- removed L7: 8.2n, Inductor_SMD:L_0603_1608Metric
- removed L8: 8.7n, Inductor_SMD:L_0603_1608Metric
- removed the R6 at (70.1, 78.9)
- added C6: 1u, Capacitor_SMD:C_0603_1608Metric, F.Cu at (105.1, 73.8)
- added C8: 0.1u, Capacitor_SMD:C_0603_1608Metric, F.Cu at (78.0, 71.1)
- C7: value 0.47u -> 4.7u
- L1: value 15u -> 10u; footprint Inductor_SMD:L_0805_2012Metric -> Inductor_SMD:L_Changjiang_FNR6028S
- U1: value STM32WLE5C8Ux -> AK09918C; footprint Package_DFN_QFN:QFN-48-1EP_7x7mm_P0.5mm_EP5.6x5.6mm -> AK09918C:BGA4_WL-CSP_AKM
- U4: value AK09918C -> STM32L431CCTx; footprint AK09918C:BGA4_WL-CSP_AKM -> Package_QFP:LQFP-48_7x7mm_P0.5mm
- moved R4 18.0 mm to (82.9, 77.8), turned to 0 degrees
- moved R5 17.8 mm to (82.9, 75.8), turned to 0 degrees
- moved C7 17.7 mm to (78.2, 63.7), turned to 90 degrees
- moved NMOS1 17.3 mm to (83.0, 80.3), turned to 180 degrees
- moved C9 15.8 mm to (80.1, 63.7), turned to 90 degrees
- moved U4 13.3 mm to (84.7, 69.2), turned to 180 degrees
- moved U1 12.6 mm to (97.7, 71.8), turned to 90 degrees
- moved R6 11.9 mm to (76.7, 80.5), turned to -90 degrees
- moved NMOS2 10.0 mm to (79.5, 80.3), turned to 180 degrees
- moved LED1 9.97 mm to (78.6, 76.8), turned to 180 degrees
- moved L1 8.45 mm to (92.1, 77.7), turned to 90 degrees
- moved C11 5.57 mm to (91.7, 72.7), turned to -90 degrees
- moved C10 4.01 mm to (93.5, 72.7), turned to -90 degrees
- moved FB1 1.78 mm to (95.5, 72.7)
- moved C3 0.13 mm to (98.2, 73.7), turned to 0 degrees
- renumbered C9 to C1, C6 to C10, C4 to C11, C8 to C2, C10 to C3, C11 to C4, C12 to C5, C3 to C9, R2 to R1, R7 to R2, R8 to R3, R3 to R4, R4 to R5, R5 to R6, R1 to R7
Connections:
- C7 pad 1: /VDDRF1V55 -> VDD
- J2 pad 3: unconnected-(J2-Pin_3-Pad3) -> VCC
- J2 pad 4: unconnected-(J2-Pin_4-Pad4) -> VDD
- L1 pad 1: /VLXSMPS -> Net-(U2-SW)
- L1 pad 2: /VDDRF1V55 -> VDD
- NMOS2 pad 3: /RF_nCTRL -> unconnected-(NMOS2-D2-Pad3)
- NMOS2 pad 4: GND -> unconnected-(NMOS2-S2-Pad4)
- NMOS2 pad 5: /RF_CTRL -> unconnected-(NMOS2-G2-Pad5)
Routing:
- net /RF_CTRL: track 36.8 -> 0.00 mm, vias 2 -> 0
- net /RFO_HP: track 33.7 -> 0.00 mm, vias 2 -> 0
- net GND: track 84.4 -> 54.3 mm, vias 24 -> 15
- net /MCU_LED_R: track 43.0 -> 17.4 mm
- net VCC: track 41.5 -> 66.5 mm, vias 0 -> 1
- net /VDDRF1V55: track 24.2 -> 0.00 mm, vias 3 -> 0
- net /VR_PA: track 20.9 -> 0.00 mm, vias 2 -> 0
- net /RF_nCTRL: track 16.0 -> 0.00 mm, vias 2 -> 0
- net /SWDIO: track 40.9 -> 55.5 mm, vias 1 -> 2
- net /LED_B: track 16.6 -> 2.76 mm, vias 2 -> 0
- net /NRST: track 46.3 -> 33.9 mm
- net /SWCLK: track 38.7 -> 50.5 mm, vias 1 -> 2
- net /RFI_P: track 10.6 -> 0.00 mm, vias 2 -> 0
- net /RF/RF_RX: track 8.85 -> 0.00 mm
- net /SDA: track 33.1 -> 41.3 mm
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Other:
- board size 51.1 x 26.9 mm -> 41.4 x 27.9 mm
- board text added: "1.8V"
- board text added: "IMU Geolocator - Loraless v0.1"
- board text added: "VCC"
- board text removed: "IMU Geolocator v0.1"

Commit message: version 0.1-loraless finished
Connections:
- J2 pad 7: /UART_RX -> /UART_TX
- J2 pad 8: /UART_TX -> /UART_RX
- U4 pad 42: /UART_RX -> /UART_TX
- U4 pad 43: /UART_TX -> /UART_RX
Routing:
- net /SWCLK: track 50.5 -> 48.5 mm
- net /SWDIO: track 55.5 -> 53.5 mm
- net /MCU_LED_B: track 29.0 -> 30.4 mm
- net +BATT: track 4.72 -> 5.99 mm, vias 1 -> 2
- net /UART_TX: track 21.0 -> 22.0 mm
- net /UART_RX: track 22.0 -> 21.0 mm
- net /MCU_LED_G: track 26.6 -> 25.7 mm
- net VDD: track 46.0 -> 46.8 mm
- net GND: track 54.3 -> 54.9 mm
- net VCC: track 66.5 -> 67.0 mm
Other:
- board text added: "IMU GL-LL v0.1"
- board text removed: "IMU Geolocator - Loraless v0.1"
